File: elec/PCA9685/PCA9685.sch (KiCad schematic (older format))
At the start: 17 parts, among them J1 Conn_bat_power, J10 Servo 2.3, J2 I2C_main_card, J3 Servo 1.1, J4 Servo 1.2, J5 Servo 1.3, J6 Servo Flag, J7 Servo Manche, J8 Servo 2.1, J9 Servo 2.2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

Commit message: Patch footprint connecteurs servo sur carte PAC9685
Parts:
- J10, J3, J4, J5, J6, J7, J8, J9: footprint Connector_JST:JST_XH_B3B-XH-A_1x03_P2.50mm_Vertical -> Connector_PinHeader_2.54mm:PinHeader_1x03_P2.54mm_Vertical
Changed lines of the file:
@@
 F 0 "J3" H 9172 1424 50  0000 R CNN
 F 1 "Servo 1.1" H 9172 1333 50  0000 R CNN
-F 2 "Connector_JST:JST_XH_B3B-XH-A_1x03_P2.50mm_Vertical" H 9200 1400 50  0001 C CNN
+F 2 "Connector_PinHeader_2.54mm:PinHeader_1x03_P2.54mm_Vertical" H 9200 1400 50  0001 C CNN
 F 3 "~" H 9200 1400 50  0001 C CNN
 	1    9200 1400
@@
 F 0 "J4" H 9172 1924 50  0000 R CNN
 F 1 "Servo 1.2" H 9172 1833 50  0000 R CNN
-F 2 "Connector_JST:JST_XH_B3B-XH-A_1x03_P2.50mm_Vertical" H 9200 1900 50  0001 C CNN
+F 2 "Connector_PinHeader_2.54mm:PinHeader_1x03_P2.54mm_Vertical" H 9200 1900 50  0001 C CNN
 F 3 "~" H 9200 1900 50  0001 C CNN
 	1    9200 1900
@@
 F 0 "J5" H 9172 2424 50  0000 R CNN
 F 1 "Servo 1.3" H 9172 2333 50  0000 R CNN
-F 2 "Connector_JST:JST_XH_B3B-XH-A_1x03_P2.50mm_Vertical" H 9200 2400 50  0001 C CNN
+F 2 "Connector_PinHeader_2.54mm:PinHeader_1x03_P2.54mm_Vertical" H 9200 2400 50  0001 C CNN
 F 3 "~" H 9200 2400 50  0001 C CNN
 	1    9200 2400
@@
 F 0 "J8" H 9172 4924 50  0000 R CNN
 F 1 "Servo 2.1" H 9172 4833 50  0000 R CNN
-F 2 "Connector_JST:JST_XH_B3B-XH-A_1x03_P2.50mm_Vertical" H 9200 4900 50  0001 C CNN
+F 2 "Connector_PinHeader_2.54mm:PinHeader_1x03_P2.54mm_Vertical" H 9200 4900 50  0001 C CNN
 F 3 "~" H 9200 4900 50  0001 C CNN
 	1    9200 4900
@@
 F 0 "J9" H 9172 5424 50  0000 R CNN
 F 1 "Servo 2.2" H 9172 5333 50  0000 R CNN
-F 2 "Connector_JST:JST_XH_B3B-XH-A_1x03_P2.50mm_Vertical" H 9200 5400 50  0001 C CNN
+F 2 "Connector_PinHeader_2.54mm:PinHeader_1x03_P2.54mm_Vertical" H 9200 5400 50  0001 C CNN
 F 3 "~" H 9200 5400 50  0001 C CNN
 	1    9200 5400
@@
 F 0 "J10" H 9172 5924 50  0000 R CNN
 F 1 "Servo 2.3" H 9172 5833 50  0000 R CNN
-F 2 "Connector_JST:JST_XH_B3B-XH-A_1x03_P2.50mm_Vertical" H 9200 5900 50  0001 C CNN
+F 2 "Connector_PinHeader_2.54mm:PinHeader_1x03_P2.54mm_Vertical" H 9200 5900 50  0001 C CNN
 F 3 "~" H 9200 5900 50  0001 C CNN
 	1    9200 5900
@@
 F 0 "J6" H 9172 3274 50  0000 R CNN
 F 1 "Servo Flag" H 9172 3183 50  0000 R CNN
-F 2 "Connector_JST:JST_XH_B3B-XH-A_1x03_P2.50mm_Vertical" H 9200 3250 50  0001 C CNN
+F 2 "Connector_PinHeader_2.54mm:PinHeader_1x03_P2.54mm_Vertical" H 9200 3250 50  0001 C CNN
 F 3 "~" H 9200 3250 50  0001 C CNN
 	1    9200 3250
@@
 F 0 "J7" H 9172 3774 50  0000 R CNN
 F 1 "Servo Manche" H 9172 3683 50  0000 R CNN
-F 2 "Connector_JST:JST_XH_B3B-XH-A_1x03_P2.50mm_Vertical" H 9200 3750 50  0001 C CNN
+F 2 "Connector_PinHeader_2.54mm:PinHeader_1x03_P2.54mm_Vertical" H 9200 3750 50  0001 C CNN
 F 3 "~" H 9200 3750 50  0001 C CNN
 	1    9200 3750
@@
 Connection ~ 3450 3450
 $Comp
-L power:+5V #PWR?
+L power:+5V #PWR0104
 U 1 1 6048A23A
 P 8750 1900
-F 0 "#PWR?" H 8750 1750 50  0001 C CNN
+F 0 "#PWR0104" H 8750 1750 50  0001 C CNN
 F 1 "+5V" V 8765 2073 50  0000 C CNN
 F 2 "" H 8750 1900 50  0001 C CNN
@@
 $EndComp
 $Comp
-L power:GND #PWR?
+L power:GND #PWR0111
 U 1 1 6048A240
 P 8650 1800
-F 0 "#PWR?" H 8650 1550 50  0001 C CNN
+F 0 "#PWR0111" H 8650 1550 50  0001 C CNN
 F 1 "GND" V 8655 1672 50  0000 R CNN
 F 2 "" H 8650 1800 50  0001 C CNN
@@
 servo1.3
 $Comp
-L power:+5V #PWR?
+L power:+5V #PWR0112
 U 1 1 6049F9B1
 P 8750 2400
-F 0 "#PWR?" H 8750 2250 50  0001 C CNN
+F 0 "#PWR0112" H 8750 2250 50  0001 C CNN
 F 1 "+5V" V 8765 2573 50  0000 C CNN
 F 2 "" H 8750 2400 50  0001 C CNN
@@
 $EndComp
 $Comp
-L power:GND #PWR?
+L power:GND #PWR0113
 U 1 1 6049F9B7
 P 8650 2300
-F 0 "#PWR?" H 8650 2050 50  0001 C CNN
+F 0 "#PWR0113" H 8650 2050 50  0001 C CNN
 F 1 "GND" V 8655 2172 50  0000 R CNN
 F 2 "" H 8650 2300 50  0001 C CNN
@@
 	9000 2400 8750 2400
 $Comp
-L power:+5V #PWR?
+L power:+5V #PWR0114
 U 1 1 604A196E
 P 8750 3250
-F 0 "#PWR?" H 8750 3100 50  0001 C CNN
+F 0 "#PWR0114" H 8750 3100 50  0001 C CNN
 F 1 "+5V" V 8765 3423 50  0000 C CNN
 F 2 "" H 8750 3250 50  0001 C CNN
@@
 $EndComp
 $Comp
-L power:GND #PWR?
+L power:GND #PWR0115
 U 1 1 604A1974
 P 8650 3150
-F 0 "#PWR?" H 8650 2900 50  0001 C CNN
+F 0 "#PWR0115" H 8650 2900 50  0001 C CNN
 F 1 "GND" V 8655 3022 50  0000 R CNN
 F 2 "" H 8650 3150 50  0001 C CNN
@@
 	9000 3250 8750 3250
 $Comp
-L power:+5V #PWR?
+L power:+5V #PWR0116
 U 1 1 604A3DF6
 P 8750 3750
-F 0 "#PWR?" H 8750 3600 50  0001 C CNN
+F 0 "#PWR0116" H 8750 3600 50  0001 C CNN
 F 1 "+5V" V 8765 3923 50  0000 C CNN
 F 2 "" H 8750 3750 50  0001 C CNN
@@
 $EndComp
 $Comp
-L power:GND #PWR?
+L power:GND #PWR0117
 U 1 1 604A3DFC
 P 8650 3650
-F 0 "#PWR?" H 8650 3400 50  0001 C CNN
+F 0 "#PWR0117" H 8650 3400 50  0001 C CNN
 F 1 "GND" V 8655 3522 50  0000 R CNN
 F 2 "" H 8650 3650 50  0001 C CNN
@@
 	9000 3750 8750 3750
 $Comp
-L power:+5V #PWR?
+L power:+5V #PWR0118
 U 1 1 604A88C9
 P 8750 4900
-F 0 "#PWR?" H 8750 4750 50  0001 C CNN
+F 0 "#PWR0118" H 8750 4750 50  0001 C CNN
 F 1 "+5V" V 8765 5073 50  0000 C CNN
 F 2 "" H 8750 4900 50  0001 C CNN
@@
 $EndComp
 $Comp
-L power:GND #PWR?
+L power:GND #PWR0119
 U 1 1 604A88CF
 P 8650 4800
-F 0 "#PWR?" H 8650 4550 50  0001 C CNN
+F 0 "#PWR0119" H 8650 4550 50  0001 C CNN
 F 1 "GND" V 8655 4672 50  0000 R CNN
 F 2 "" H 8650 4800 50  0001 C CNN
@@
 	9000 4900 8750 4900
 $Comp
-L power:+5V #PWR?
+L power:+5V #PWR0120
 U 1 1 604AB7A3
 P 8750 5400
-F 0 "#PWR?" H 8750 5250 50  0001 C CNN
+F 0 "#PWR0120" H 8750 5250 50  0001 C CNN
 F 1 "+5V" V 8765 5573 50  0000 C CNN
 F 2 "" H 8750 5400 50  0001 C CNN
@@
 $EndComp
 $Comp
-L power:GND #PWR?
+L power:GND #PWR0121
 U 1 1 604AB7A9
 P 8650 5300
-F 0 "#PWR?" H 8650 5050 50  0001 C CNN
+F 0 "#PWR0121" H 8650 5050 50  0001 C CNN
 F 1 "GND" V 8655 5172 50  0000 R CNN
 F 2 "" H 8650 5300 50  0001 C CNN
@@
 	9000 5400 8750 5400
 $Comp
-L power:+5V #PWR?
+L power:+5V #PWR0122
 U 1 1 604AD8DA
 P 8750 5900
-F 0 "#PWR?" H 8750 5750 50  0001 C CNN
+F 0 "#PWR0122" H 8750 5750 50  0001 C CNN
 F 1 "+5V" V 8765 6073 50  0000 C CNN
 F 2 "" H 8750 5900 50  0001 C CNN
@@
 $EndComp
 $Comp
-L power:GND #PWR?
+L power:GND #PWR0123
 U 1 1 604AD8E0
 P 8650 5800
-F 0 "#PWR?" H 8650 5550 50  0001 C CNN
+F 0 "#PWR0123" H 8650 5550 50  0001 C CNN
 F 1 "GND" V 8655 5672 50  0000 R CNN
 F 2 "" H 8650 5800 50  0001 C CNN
