File: elec/pcb_robot_2021A/pcb_robot_2021A.kicad_pcb (KiCad board)
At the start: 2 copper layers, 99 x 79 mm, 43 parts, among them J1 LCD, J10 Encodeur 1, J11 Encodeur 2, J12 Conn_bat_pwr, J13 Tirette, J14 Couleur, J15 UART_backup, J16 Xbee, J17 PCA9685, J18 Capt_US, J19 I2C_backup, J2 IR 1.1, J20 lidar in, J21 lidar_out, J22 Lidar alim, J23 Galet 1.1, J24 Galet 1.2, J25 Galet 2.1, J26 Galet 2.2, J3 IR 1.2, J4 IR 1.3, J5 IR 2.1, J6 IR 2.2, J7 IR 2.3, J8 Moteur 1, J9 Moteur 2, U1 R-78E5.0-1.0, U2 Teensy3.5, U3 mosfet_lid_I1, U4 mosfet_lid_I2, U5 mosfet_lid_I3, U6 mosfet_lid_I4, U7 mosfet_lid_I5

Commit message: Final push
Changed lines of the file:
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@@
       (plotvalue true)
       (plotinvisibletext false)
-      (padsonsilk false)
+      (padsonsilk true)
       (subtractmaskfromsilk false)
       (outputformat 1)
       (mirror false)
-      (drillshape 1)
+      (drillshape 0)
       (scaleselection 1)
-      (outputdirectory ""))
+      (outputdirectory "gerbers/"))
   )
   (net 0 "")
@@
       (effects (font (size 1 1) (thickness 0.15)))
     )
-    (fp_text value "IR 1.3" (at 3 -3.5 90) (layer F.SilkS)
+    (fp_text value "IR 1.3" (at 2.5 4.5 90) (layer F.SilkS)
       (effects (font (size 0.8 1) (thickness 0.15)))
     )
@@
       (effects (font (size 1 1) (thickness 0.15)))
     )
-    (fp_text value "IR 1.2" (at 3 -3.5 90) (layer F.SilkS)
+    (fp_text value "IR 1.2" (at 3 4.5 90) (layer F.SilkS)
       (effects (font (size 0.8 1) (thickness 0.15)))
     )
@@
       (effects (font (size 1 1) (thickness 0.15)))
     )
-    (fp_text value "IR 1.1" (at 2.5 -3.5 90) (layer F.SilkS)
-      (effects (font (size 0.8 1) (thickness 0.15)))
-    )
+    (fp_text value "IR 1.1" (at 3 4.5 90) (layer F.SilkS)
+      (effects (font (size 0.8 1) (thickness 0.15)))
+    )
